Commit message: [dev] fix bug

File: src/rm_bringup/src/urdf/shaobing.urdf (robot description, URDF)
Before this commit: robot sam_bot, 7 links, 6 joints
Joints:
- joint base_joint: child livox_frame -> base_link; parent base_link -> livox_frame

File: src/rm_bringup/src/urdf/test.urdf (robot description, URDF)
Before this commit: robot sentry, 5 links, 4 joints
Joints:
- joint base_joint: origin xyz=-0.105 0 -0.460 rpy=0 0 0 -> xyz=-0.105 0 -0.460 rpy=0 0 ${pi}
