Commit message: 1.14

File: src/rm_bringup/src/urdf/test.urdf (robot description, URDF)
Before this commit: robot sentry, 5 links, 4 joints
Joints:
- joint base_joint: origin xyz=-0.105 0 -0.460 rpy=0 0 ${pi} -> xyz=0.0 0.135 -0.20 rpy=0 ${-pi/4} 0

Commit message: 3.9

File: src/rm_bringup/src/urdf/test.urdf (robot description, URDF)
Before this commit: robot sentry, 5 links, 4 joints
Joints:
- joint base_joint: origin xyz=0.0 0.135 -0.20 rpy=0 ${-pi/4} 0 -> xyz=0.0 0.135 -0.20 rpy=${pi} 0 0

File: src/rm_gimbal_description/urdf/rm_gimbal.urdf.xacro (robot description, xacro)
@@ -2,6 +2,4 @@
 <robot name="rm_gimbal"
   xmlns:xacro="http://ros.org/wiki/xacro">
-  <xacro:arg name="xyz" default="0.00 0.00 0.040" />
-  <xacro:arg name="rpy" default="0 ${pi/2} 0" />
   <link name="odom" />
   <link name="gimbal_link" />
@@ -12,5 +10,5 @@
   <link name="camera_link" />
   <joint name="camera_joint" type="fixed">
-    <origin xyz="$(arg xyz)" rpy="$(arg rpy)" />
+    <origin xyz="0.080 0.000 0.04" rpy="0 0.0 ${pi/32}" />
     <parent link="gimbal_link" />
     <child link="camera_link" />
@@ -23,3 +21,8 @@
     <child link="camera_optical_frame" />
   </joint>
+  <link name="horizom_gimbal_link" />
+  <joint name="horizom_gimbal_joint" type="floating">
+    <parent link = "gimbal_link" />
+    <child link = "horizom_gimbal_link" />
+  </joint>
 </robot>
